File: arisu.kicad_pcb (KiCad board)
At the start: 2 copper layers, 339.1 x 118.7 mm, 176 parts, among them J1 USB_B_Micro, SW1 SW_Push, SW10 SW_Push, SW11 SW_Push, SW12 SW_Push, SW13 SW_Push, SW14 SW_Push, SW15 SW_Push, SW16 SW_Push, SW17 SW_Push, SW18 SW_Push, SW19 SW_Push, SW2 SW_Push, SW20 SW_Push, SW21 SW_Push, SW22 SW_Push, SW23 SW_Push, SW24 SW_Push, SW25 SW_Push, SW26 SW_Push, SW27 SW_Push, SW28 SW_Push, SW29 SW_Push, SW3 SW_Push, SW30 SW_Push, SW31 SW_Push, SW32 SW_Push, SW33 SW_Push, SW34 SW_Push, SW35 SW_Push, SW36 SW_Push, SW37 SW_Push, SW38 SW_Push, SW39 SW_Push, SW4 SW_Push, SW40 SW_Push, SW41 SW_Push, SW42 SW_Push, SW43 SW_Push, SW44 SW_Push, SW45 SW_Push, SW46 SW_Push, SW47 SW_Push, SW48 SW_Push, SW49 SW_Push, SW5 SW_Push, SW50 SW_Push, SW51 SW_Push, SW52 SW_Push, SW53 SW_Push, SW54 SW_Push, SW55 SW_Push, SW56 SW_Push, SW57 SW_Push, SW58 SW_Push, SW59 SW_Push, SW6 SW_Push, SW60 SW_Push, SW61 SW_Push, SW62 SW_Push, SW63 SW_Push, SW64 SW_Push, SW65 SW_Push, SW66 SW_Push, SW67 SW_Push, SW7 SW_Push, SW8 SW_Push, SW9 SW_Push, U1 USBLC6-2SC6, U2 ATmega32U4-AU, Y1 Crystal_GND24

Commit message: got rid of the MCU and added a pro micro
Parts:
- removed C1, C2: 22pF, Capacitors_SMD:C_0805_HandSoldering
- removed C3: 10uF, Capacitors_SMD:C_0805_HandSoldering
- removed C4: 1uF (±10%), Capacitors_SMD:C_0805_HandSoldering
- removed C5: 1uF, Capacitors_SMD:C_0805_HandSoldering
- removed C6, C7, C8, C9: 0.1uF, Capacitors_SMD:C_0805_HandSoldering
- removed D+: D+, Pin_Headers:Pin_Header_Straight_1x01_Pitch2.54mm
- removed D-: D-, Pin_Headers:Pin_Header_Straight_1x01_Pitch2.54mm
- removed G*** (x2): LOGO, arisu:arisu-logo
- removed GND (x2): GND, Pin_Headers:Pin_Header_Straight_1x01_Pitch2.54mm
- removed H1, H2, H3, H4, H5, H6, H7, H8: MountingHole, Mounting_Holes:MountingHole_2.2mm_M2_Pad
- removed J1: USB_B_Micro, Connectors_USB:USB_Micro-B_Molex-105017-0001
- removed MISO: MISO, Pin_Headers:Pin_Header_Straight_1x01_Pitch2.54mm
- removed MOSI: MOSI, Pin_Headers:Pin_Header_Straight_1x01_Pitch2.54mm
- removed PF4: PF4, Pin_Headers:Pin_Header_Straight_1x01_Pitch2.54mm
- removed PF5: PF5, Pin_Headers:Pin_Header_Straight_1x01_Pitch2.54mm
- removed PF6: PF6, Pin_Headers:Pin_Header_Straight_1x01_Pitch2.54mm
- removed PF7: PF7, Pin_Headers:Pin_Header_Straight_1x01_Pitch2.54mm
- removed R1, R2: 22, Resistors_SMD:R_0805_HandSoldering
- removed R3, R4: 10K, Resistors_SMD:R_0805_HandSoldering
- removed RES: RES, Pin_Headers:Pin_Header_Straight_1x01_Pitch2.54mm
- removed SCK: SCK, Pin_Headers:Pin_Header_Straight_1x01_Pitch2.54mm
- removed SWR1: SW_Push, Buttons_Switches_SMD:SW_SPST_TL3342
- removed U2: ATmega32U4-AU, Housings_QFP:TQFP-44_10x10mm_Pitch0.8mm
- removed VCC (x2): VCC, Pin_Headers:Pin_Header_Straight_1x01_Pitch2.54mm
- removed Y1: Crystal_GND24, Crystals:Crystal_SMD_SeikoEpson_FA238-4pin_3.2x2.5mm_HandSoldering
- U1: value USBLC6-2SC6 -> ProMicro; footprint TO_SOT_Packages_SMD:SOT-23-6_Handsoldering -> Keebio-Parts:ArduinoProMicro; moved to F.Cu
- moved U1 9.44 mm to (175.7, 27.8), turned to 270 degrees
Connections:
- net /col13 renamed /matrix/col13
- net /col2 renamed /matrix/col2
- net /col9 renamed /matrix/col9
- net /row3 renamed /matrix/row3
- D1 pad 1: /row0 -> /matrix/row0
- D10 pad 1: /row0 -> /matrix/row0
- D11 pad 1: /row1 -> /matrix/row1
- D12 pad 1: /row2 -> /matrix/row1
- D14 pad 1: /row4 -> /matrix/row4
- D15 pad 1: /row0 -> /matrix/row0
- D16 pad 1: /row1 -> /matrix/row1
- D17 pad 1: /row2 -> /matrix/row1
- D19 pad 1: /row0 -> /matrix/row0
- D2 pad 1: /row1 -> /matrix/row1
- D20 pad 1: /row1 -> /matrix/row1
- D21 pad 1: /row2 -> /matrix/row1
- D23 pad 1: /row4 -> /matrix/row4
- D24 pad 1: /row0 -> /matrix/row0
- D25 pad 1: /row1 -> /matrix/row1
- D26 pad 1: /row2 -> /matrix/row1
- D28 pad 1: /row4 -> /matrix/row4
- D29 pad 1: /row0 -> /matrix/row0
- D3 pad 1: /row2 -> /matrix/row1
- D30 pad 1: /row1 -> /matrix/row1
- D31 pad 1: /row2 -> /matrix/row1
- D33 pad 1: /row0 -> /matrix/row0
- D34 pad 1: /row1 -> /matrix/row1
- D35 pad 1: /row2 -> /matrix/row1
- D37 pad 1: /row4 -> /matrix/row4
- D38 pad 1: /row0 -> /matrix/row0
- D39 pad 1: /row1 -> /matrix/row1
- D40 pad 1: /row2 -> /matrix/row1
- D42 pad 1: /row0 -> /matrix/row0
- D43 pad 1: /row1 -> /matrix/row1
- D44 pad 1: /row2 -> /matrix/row1
- D46 pad 1: /row4 -> /matrix/row4
- D47 pad 1: /row0 -> /matrix/row0
- D48 pad 1: /row1 -> /matrix/row1
- D49 pad 1: /row2 -> /matrix/row1
- D5 pad 1: /row4 -> /matrix/row4
- D51 pad 1: /row0 -> /matrix/row0
- D52 pad 1: /row1 -> /matrix/row1
- D53 pad 1: /row2 -> /matrix/row1
- D55 pad 1: /row0 -> /matrix/row0
- D56 pad 1: /row1 -> /matrix/row1
- D57 pad 1: /row2 -> /matrix/row1
- D58 pad 1: /row4 -> /matrix/row4
- D59 pad 1: /row0 -> /matrix/row0
- D6 pad 1: /row0 -> /matrix/row0
- D60 pad 1: /row1 -> /matrix/row1
- D62 pad 1: /row4 -> /matrix/row4
- D63 pad 1: /row0 -> /matrix/row0
- D64 pad 1: /row1 -> /matrix/row1
- D65 pad 1: /row2 -> /matrix/row1
- D67 pad 1: /row4 -> /matrix/row4
- D7 pad 1: /row1 -> /matrix/row1
- D8 pad 1: /row2 -> /matrix/row1
- SW1 pad 1: /col0 -> /matrix/col0
- SW15 pad 1: /col3 -> /matrix/col3
- SW16 pad 1: /col3 -> /matrix/col3
- SW17 pad 1: /col3 -> /matrix/col3
- SW18 pad 1: /col3 -> /matrix/col3
- SW19 pad 1: /col4 -> /matrix/col4
- SW2 pad 1: /col0 -> /matrix/col0
- SW20 pad 1: /col4 -> /matrix/col4
- SW21 pad 1: /col4 -> /matrix/col4
- SW22 pad 1: /col4 -> /matrix/col4
- SW23 pad 1: /col4 -> /matrix/col4
- SW24 pad 1: /col5 -> /matrix/col4
- SW25 pad 1: /col5 -> /matrix/col4
- SW26 pad 1: /col5 -> /matrix/col4
- SW27 pad 1: /col5 -> /matrix/col4
- SW28 pad 1: /col5 -> /matrix/col4
- SW29 pad 1: /col6 -> /matrix/col6
- SW3 pad 1: /col0 -> /matrix/col0
- SW30 pad 1: /col6 -> /matrix/col6
- SW31 pad 1: /col6 -> /matrix/col6
- SW32 pad 1: /col6 -> /matrix/col6
- SW33 pad 1: /SCK -> /matrix/col6
- SW34 pad 1: /SCK -> /matrix/col6
- SW35 pad 1: /SCK -> /matrix/col6
- SW36 pad 1: /SCK -> /matrix/col6
- SW37 pad 1: /SCK -> /matrix/col6
- SW38 pad 1: /col8 -> /matrix/col8
- SW39 pad 1: /col8 -> /matrix/col8
- SW4 pad 1: /col0 -> /matrix/col0
- SW40 pad 1: /col8 -> /matrix/col8
- SW41 pad 1: /col8 -> /matrix/col8
- SW47 pad 1: /col10 -> /matrix/col10
- SW48 pad 1: /col10 -> /matrix/col10
- SW49 pad 1: /col10 -> /matrix/col10
- SW5 pad 1: /col0 -> /matrix/col0
- SW50 pad 1: /col10 -> /matrix/col10
- SW51 pad 1: /col11 -> /matrix/col10
- SW52 pad 1: /col11 -> /matrix/col10
- SW53 pad 1: /col11 -> /matrix/col10
- SW54 pad 1: /col11 -> /matrix/col10
- SW55 pad 1: /col12 -> /matrix/col12
- SW56 pad 1: /col12 -> /matrix/col12
- SW57 pad 1: /col12 -> /matrix/col12
- SW58 pad 1: /col12 -> /matrix/col12
- SW6 pad 1: /col1 -> /matrix/col0
- SW63 pad 1: /MISO -> /matrix/col14
- SW64 pad 1: /MISO -> /matrix/col14
- SW65 pad 1: /MISO -> /matrix/col14
- SW66 pad 1: /MISO -> /matrix/col14
- SW67 pad 1: /MISO -> /matrix/col14
- SW7 pad 1: /col1 -> /matrix/col0
- SW8 pad 1: /col1 -> /matrix/col0
- SW9 pad 1: /col1 -> /matrix/col0
- U1 pad 2: GND -> Net-(U1-Pad2)
- U1 pad 5: VCC -> /matrix/col14
- U1 pad 6: Net-(J1-Pad3) -> /matrix/col12
Routing:
- net /row4: track 433.8 -> 0.00 mm, vias 2 -> 0
- net /matrix/row3: track 432.5 -> 0.00 mm, vias 2 -> 0
- net /row2: track 399.4 -> 0.00 mm, vias 4 -> 0
- net /row1: track 384.1 -> 0.00 mm, vias 4 -> 0
- net /row0: track 328.0 -> 0.00 mm, vias 4 -> 0
- net /MISO: track 272.2 -> 0.00 mm, vias 1 -> 0
- net /matrix/col13: track 269.0 -> 0.00 mm
- net /col12: track 249.0 -> 0.00 mm
- net /col11: track 230.6 -> 0.00 mm
- net /col10: track 221.3 -> 0.00 mm
- net VCC: track 205.4 -> 0.00 mm, vias 9 -> 0
- net /col0: track 204.4 -> 0.00 mm
- net /matrix/col2: track 175.7 -> 0.00 mm, vias 2 -> 0
- net /col1: track 166.8 -> 0.00 mm
- net /SCK: track 157.0 -> 0.00 mm, vias 2 -> 0
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